Commit message: Intenté desarrollar el RRT aerial y el robot aerial

File: hybrid_robot_ws/src/hybrid_robot_description/urdf/hybrid_aerial.xacro (robot description, xacro)
@@ -4,33 +4,23 @@
         <link name="drone_base_link">
             <visual>
-                <origin xyz="0 0 0.025" rpy="0 0 0" />
-                <geometry><box size="0.3 0.3 0.05" /></geometry>
-                <material name="Blue"><color rgba="0 0 1 1"/></material>
+                <origin xyz="0 0 0.025" rpy="0 0 0" /><geometry><box size="0.3 0.3 0.05" /></geometry><material name="Blue"/>
             </visual>
-            <collision>
-                <origin xyz="0 0 0.025" rpy="0 0 0" />
-                <geometry><box size="0.3 0.3 0.05" /></geometry>
-            </collision>
+            <collision><origin xyz="0 0 0.025" rpy="0 0 0" /><geometry><box size="0.3 0.3 0.05" /></geometry></collision>
             <inertial>
-                <mass value="1.0" />
+                <mass value="0.5" />
                 <inertia ixx="0.01" ixy="0" ixz="0" iyy="0.01" iyz="0" izz="0.02" />
             </inertial>
         </link>
-        <joint name="drone_to_terrestrial_joint" type="fixed">
-            <parent link="${parent_link}" />
-            <child link="drone_base_link" />
-            <origin xyz="0 0 0.01" rpy="0 0 0" />
+        <joint name="drone_to_terrestrial_joint" type="prismatic">
+            <parent link="${parent_link}" /><child link="drone_base_link" />
+            <origin xyz="0 0 0.01" rpy="0 0 0" /><axis xyz="0 0 1" />
+            <limit lower="0" upper="3.0" effort="2000" velocity="1.0" />
+            <dynamics damping="100.0" friction="50.0"/>
         </joint>
         <xacro:macro name="prop" params="p_name x y">
-            <link name="${p_name}_link">
-                <visual><geometry><cylinder radius="0.08" length="0.01"/></geometry></visual>
-            </link>
-            <joint name="${p_name}_joint" type="fixed">
-                <parent link="drone_base_link"/><child link="${p_name}_link"/>
-                <origin xyz="${x} ${y} 0.05" rpy="0 0 0"/>
-            </joint>
+            <link name="${p_name}_link"><visual><geometry><cylinder radius="0.08" length="0.01"/></geometry></visual></link>
+            <joint name="${p_name}_joint" type="fixed"><parent link="drone_base_link"/><child link="${p_name}_link"/><origin xyz="${x} ${y} 0.05" rpy="0 0 0"/></joint>
         </xacro:macro>
-        <xacro:prop p_name="fl" x="0.12" y="0.12"/><xacro:prop p_name="fr" x="0.12" y="-0.12"/>
-        <xacro:prop p_name="rl" x="-0.12" y="0.12"/><xacro:prop p_name="rr" x="-0.12" y="-0.12"/>
+        <xacro:prop p_name="fl" x="0.12" y="0.12"/><xacro:prop p_name="fr" x="0.12" y="-0.12"/><xacro:prop p_name="rl" x="-0.12" y="0.12"/><xacro:prop p_name="rr" x="-0.12" y="-0.12"/>
     </xacro:macro>
 </robot>

File: hybrid_robot_ws/src/hybrid_robot_description/urdf/hybrid_terrestrial.xacro (robot description, xacro)
@@ -3,5 +3,5 @@
     <xacro:property name="wheel_radius" value="0.1" />
     <xacro:property name="base_height" value="0.1" />
-    <xacro:property name="base_mass" value="5.0" />
+    <xacro:property name="base_mass" value="1.0" />
     <xacro:property name="base_length" value="0.8" />
     <xacro:property name="base_width" value="0.6" />
@@ -28,5 +28,5 @@
         <xacro:default_inertial mass="${base_mass}"/>
     </link>
-  <xacro:macro name="wheel_link" params="prefix parent_link x_offset y_offset">
+    <xacro:macro name="wheel_link" params="prefix parent_link x_offset y_offset">
         <link name="${prefix}_wheel_link">
             <visual>
@@ -42,16 +42,10 @@
         </link>
         <gazebo reference="${prefix}_wheel_link">
-            <mu1 value="1.0"/>
-            <mu2 value="1.0"/>
-            <kp value="10000000.0" />
-            <kd value="1.0" />
-            <fdir1 value="1 0 0"/>
+            <mu1 value="1.0"/><mu2 value="1.0"/><kp value="10000000.0" /><kd value="1.0" />
             <material>Gazebo/Black</material>
         </gazebo>
         <joint name="${prefix}_wheel_joint" type="continuous">
             <origin xyz="${x_offset} ${y_offset} ${wheel_radius}" rpy="0 0 0" />
-            <parent link="${parent_link}" />
-            <child link="${prefix}_wheel_link" />
-            <axis xyz="0 1 0" />
+            <parent link="${parent_link}" /><child link="${prefix}_wheel_link" /><axis xyz="0 1 0" />
         </joint>
     </xacro:macro>
@@ -59,83 +53,54 @@
     <xacro:wheel_link prefix="right" parent_link="base_link" x_offset="0.25" y_offset="-${wheel_separation/2}" />
     <link name="caster_front_link">
-        <visual>
-            <origin xyz="0 0 0" rpy="0 0 0"/>
-            <geometry><sphere radius="${caster_radius}"/></geometry>
-            <material name="Black"/>
-        </visual>
-        <collision>
-            <origin xyz="0 0 0" rpy="0 0 0"/>
-            <geometry><sphere radius="${caster_radius}"/></geometry>
-        </collision>
+        <visual><geometry><sphere radius="${caster_radius}"/></geometry><material name="Black"/></visual>
+        <collision><geometry><sphere radius="${caster_radius}"/></geometry></collision>
         <xacro:default_inertial mass="${caster_mass}"/>
     </link>
     <joint name="caster_front_joint" type="fixed">
-        <origin xyz="${base_length/2 - caster_radius*2} 0 ${caster_radius}" rpy="0 0 0"/>
-        <parent link="base_link" />
-        <child link="caster_front_link" />
+        <origin xyz="${base_length/2 - caster_radius*2} 0 ${caster_radius}" rpy="0 0 0"/><parent link="base_link" /><child link="caster_front_link" />
     </joint>
     <link name="caster_rear_link">
-        <visual>
-            <origin xyz="0 0 0" rpy="0 0 0"/>
-            <geometry><sphere radius="${caster_radius}"/></geometry>
-            <material name="Black"/>
-        </visual>
-        <collision>
-            <origin xyz="0 0 0" rpy="0 0 0"/>
-            <geometry><sphere radius="${caster_radius}"/></geometry>
-        </collision>
+        <visual><geometry><sphere radius="${caster_radius}"/></geometry><material name="Black"/></visual>
+        <collision><geometry><sphere radius="${caster_radius}"/></geometry></collision>
         <xacro:default_inertial mass="${caster_mass}"/>
     </link>
     <joint name="caster_rear_joint" type="fixed">
-        <origin xyz="${-base_length/2 + caster_radius*2} 0 ${caster_radius}" rpy="0 0 0"/>
-        <parent link="base_link" />
-        <child link="caster_rear_link" />
+        <origin xyz="${-base_length/2 + caster_radius*2} 0 ${caster_radius}" rpy="0 0 0"/><parent link="base_link" /><child link="caster_rear_link" />
     </joint>
-    <gazebo reference="caster_front_link">
-        <mu1 value="0.001"/>
-        <mu2 value="0.001"/>
-    </gazebo>
-    <gazebo reference="caster_rear_link">
-        <mu1 value="0.001"/>
-        <mu2 value="0.001"/>
-    </gazebo>
-<xacro:include filename="hybrid_aerial.xacro" />
+    <xacro:include filename="hybrid_aerial.xacro" />
     <link name="landing_pad">
-        <visual>
-            <origin xyz="0 0 0" rpy="0 0 0" />
-            <geometry><box size="0.4 0.4 0.01" /></geometry>
-            <material name="Grey"><color rgba="0.5 0.5 0.5 1"/></material>
-        </visual>
-        <collision>
-            <origin xyz="0 0 0" rpy="0 0 0" />
-            <geometry><box size="0.4 0.4 0.01" /></geometry>
-        </collision>
+        <visual><geometry><box size="0.4 0.4 0.01" /></geometry><material name="Grey"/></visual>
+        <collision><geometry><box size="0.4 0.4 0.01" /></geometry></collision>
         <xacro:default_inertial mass="0.1"/>
     </link>
     <joint name="landing_pad_joint" type="fixed">
-        <parent link="base_link" />
-        <child link="landing_pad" />
-        <origin xyz="0 0 0.2" rpy="0 0 0" />
+        <parent link="base_link" /><child link="landing_pad" /><origin xyz="0 0 0.2" rpy="0 0 0" />
     </joint>
     <xacro:drone_assembly parent_link="landing_pad" />
+    <gazebo>
+        <plugin name="global_aerial_controller" filename="libgazebo_ros_planar_move.so">
+            <ros>
+                <remapping>cmd_vel:=drone_cmd_vel</remapping>
+                <remapping>odom:=drone_odom</remapping>
+            </ros>
+            <update_rate>100</update_rate>
+            <publish_odom>true</publish_odom>
+            <publish_odom_tf>true</publish_odom_tf>
+            <robot_base_frame>base_link</robot_base_frame>
+        </plugin>
+    </gazebo>
     <ros2_control name="TerrestrialRobot" type="system">
-        <hardware>
-            <plugin>gazebo_ros2_control/GazeboSystem</plugin>
-        </hardware>
+        <hardware><plugin>gazebo_ros2_control/GazeboSystem</plugin></hardware>
         <joint name="left_wheel_joint">
-            <command_interface name="velocity">
-                <param name="min">-10</param>
-                <param name="max">10</param>
-            </command_interface>
-            <state_interface name="velocity"/>
-            <state_interface name="position"/>
+            <command_interface name="velocity"><param name="min">-10</param><param name="max">10</param></command_interface>
+            <state_interface name="velocity"/><state_interface name="position"/>
         </joint>
         <joint name="right_wheel_joint">
-            <command_interface name="velocity">
-                <param name="min">-10</param>
-                <param name="max">10</param>
-            </command_interface>
-            <state_interface name="velocity"/>
-            <state_interface name="position"/>
+            <command_interface name="velocity"><param name="min">-10</param><param name="max">10</param></command_interface>
+            <state_interface name="velocity"/><state_interface name="position"/>
+        </joint>
+        <joint name="drone_to_terrestrial_joint">
+            <command_interface name="position"><param name="min">0</param><param name="max">5</param></command_interface>
+            <state_interface name="position"/><state_interface name="velocity"/>
         </joint>
     </ros2_control>
