Commit message: Gazebo sigue aproximadamente RVIZ en la parte terrestre con RRT

File: hybrid_robot_ws/src/hybrid_robot_description/urdf/hybrid_terrestrial.xacro (robot description, xacro)
@@ -3,5 +3,5 @@
     <xacro:property name="wheel_radius" value="0.1" />
     <xacro:property name="base_height" value="0.1" />
-    <xacro:property name="base_mass" value="10.0" />
+    <xacro:property name="base_mass" value="5.0" />
     <xacro:property name="base_length" value="0.8" />
     <xacro:property name="base_width" value="0.6" />
@@ -28,5 +28,5 @@
         <xacro:default_inertial mass="${base_mass}"/>
     </link>
-    <xacro:macro name="wheel_link" params="prefix parent_link x_offset y_offset">
+  <xacro:macro name="wheel_link" params="prefix parent_link x_offset y_offset">
         <link name="${prefix}_wheel_link">
             <visual>
@@ -41,4 +41,12 @@
             <xacro:default_inertial mass="0.5" />
         </link>
+        <gazebo reference="${prefix}_wheel_link">
+            <mu1 value="1.0"/>
+            <mu2 value="1.0"/>
+            <kp value="10000000.0" />
+            <kd value="1.0" />
+            <fdir1 value="1 0 0"/>
+            <material>Gazebo/Black</material>
+        </gazebo>
         <joint name="${prefix}_wheel_joint" type="continuous">
             <origin xyz="${x_offset} ${y_offset} ${wheel_radius}" rpy="0 0 0" />
@@ -47,7 +55,4 @@
             <axis xyz="0 1 0" />
         </joint>
-        <gazebo reference="${prefix}_wheel_link">
-          <material>Gazebo/Black</material>
-        </gazebo>
     </xacro:macro>
     <xacro:wheel_link prefix="left" parent_link="base_link" x_offset="0.25" y_offset="${wheel_separation/2}" />
@@ -87,4 +92,12 @@
         <child link="caster_rear_link" />
     </joint>
+    <gazebo reference="caster_front_link">
+        <mu1 value="0.001"/>
+        <mu2 value="0.001"/>
+    </gazebo>
+    <gazebo reference="caster_rear_link">
+        <mu1 value="0.001"/>
+        <mu2 value="0.001"/>
+    </gazebo>
 <xacro:include filename="hybrid_aerial.xacro" />
     <link name="landing_pad">

Commit message: style: green robot, fixed goal marker and renamed world files

File: hybrid_robot_ws/src/hybrid_robot_description/urdf/hybrid_terrestrial.xacro (robot description, xacro)
@@ -145,3 +145,6 @@
         </plugin>
     </gazebo>
+    <gazebo reference="base_link">
+        <material>Gazebo/Green</material>
+    </gazebo>
 </robot>
