Commit message: El RRT 2D funciona con el nuevo topic de comando que nos permitira volar y el orobot puede volar

File: hybrid_robot_ws/src/hybrid_robot_description/urdf/hybrid_robot.xacro (robot description, xacro)
@@ -3,4 +3,10 @@
     <xacro:include filename="hybrid_terrestrial.xacro" />
     <xacro:include filename="hybrid_aerial.xacro" />
+    <link name="base_footprint"/>
+    <joint name="base_footprint_joint" type="fixed">
+        <parent link="base_footprint"/>
+        <child link="world_anchor"/>
+        <origin xyz="0 0 0" rpy="0 0 0"/>
+    </joint>
     <link name="world_anchor">
         <inertial>
@@ -58,4 +64,6 @@
         <plugin name="drone_flight_controller" filename="libgazebo_ros_planar_move.so">
             <ros>
+                <namespace>/</namespace>
+                <parameter name="use_sim_time" value="true" />
                 <remapping>cmd_vel:=cmd_drone</remapping>
                 <remapping>odom:=odom_drone</remapping>

Commit message: feat: planificacion 3D que funciona con la map forest con obstaculos aereos

File: hybrid_robot_ws/src/hybrid_robot_description/urdf/hybrid_robot.xacro (robot description, xacro)
@@ -11,5 +11,5 @@
     <link name="world_anchor">
         <inertial>
-            <mass value="1.0"/>
+            <mass value="10.0"/>
             <inertia ixx="0.01" ixy="0" ixz="0" iyy="0.01" iyz="0" izz="0.01"/>
         </inertial>
