Commit message: Modification : Ahora el diff_drive_controller works. Pero todavia la teleoperacion no funciona y el aparicion del mapa en RVIZ

File: hybrid_robot_ws/install/hybrid_robot_description/share/hybrid_robot_description/urdf/hybrid_terrestrial.xacro (robot description, xacro)
@@ -87,4 +87,25 @@
         <child link="caster_rear_link" />
     </joint>
+    <ros2_control name="TerrestrialRobot" type="system">
+        <hardware>
+            <plugin>gazebo_ros2_control/GazeboSystem</plugin>
+        </hardware>
+        <joint name="left_wheel_joint">
+            <command_interface name="velocity">
+                <param name="min">-10</param>
+                <param name="max">10</param>
+            </command_interface>
+            <state_interface name="velocity"/>
+            <state_interface name="position"/>
+        </joint>
+        <joint name="right_wheel_joint">
+            <command_interface name="velocity">
+                <param name="min">-10</param>
+                <param name="max">10</param>
+            </command_interface>
+            <state_interface name="velocity"/>
+            <state_interface name="position"/>
+        </joint>
+    </ros2_control>
     <gazebo>
         <plugin filename="libgazebo_ros2_control.so" name="gazebo_ros2_control">

Commit message: Modificacion : Amelioracion fisica del robot

File: hybrid_robot_ws/install/hybrid_robot_description/share/hybrid_robot_description/urdf/hybrid_terrestrial.xacro (robot description, xacro)
@@ -18,10 +18,10 @@
     <link name="base_link">
         <visual>
-            <origin xyz="0 0 ${base_height/2}" rpy="0 0 0" />
+            <origin xyz="0 0 ${wheel_radius + base_height/2}" rpy="0 0 0" />
             <geometry><box size="${base_length} ${base_width} ${base_height}" /></geometry>
             <material name="White"><color rgba="1 1 1 1"/></material>
         </visual>
         <collision>
-            <origin xyz="0 0 ${base_height/2}" rpy="0 0 0" />
+            <origin xyz="0 0 ${wheel_radius + base_height/2}" rpy="0 0 0" />
             <geometry><box size="${base_length} ${base_width} ${base_height}" /></geometry>
         </collision>

Commit message: HE anadido el robot aereo fisico pero todavia no se mueve

File: hybrid_robot_ws/install/hybrid_robot_description/share/hybrid_robot_description/urdf/hybrid_terrestrial.xacro (robot description, xacro)
@@ -87,4 +87,23 @@
         <child link="caster_rear_link" />
     </joint>
+<xacro:include filename="hybrid_aerial.xacro" />
+    <link name="landing_pad">
+        <visual>
+            <origin xyz="0 0 0" rpy="0 0 0" />
+            <geometry><box size="0.4 0.4 0.01" /></geometry>
+            <material name="Grey"><color rgba="0.5 0.5 0.5 1"/></material>
+        </visual>
+        <collision>
+            <origin xyz="0 0 0" rpy="0 0 0" />
+            <geometry><box size="0.4 0.4 0.01" /></geometry>
+        </collision>
+        <xacro:default_inertial mass="0.1"/>
+    </link>
+    <joint name="landing_pad_joint" type="fixed">
+        <parent link="base_link" />
+        <child link="landing_pad" />
+        <origin xyz="0 0 0.2" rpy="0 0 0" />
+    </joint>
+    <xacro:drone_assembly parent_link="landing_pad" />
     <ros2_control name="TerrestrialRobot" type="system">
         <hardware>

Commit message: Stabilizacion del RRt e integracion al launch file. Aora, con el launch file, calcula la trayectoria del RRT directamente

File: hybrid_robot_ws/install/hybrid_robot_description/share/hybrid_robot_description/urdf/hybrid_terrestrial.xacro (robot description, xacro)
@@ -1,134 +1 @@
-<?xml version="1.0"?>
-<robot name="hybrid_robot_terrestrial" xmlns:xacro="http://www.ros.org/wiki/xacro">
-    <xacro:property name="wheel_radius" value="0.1" />
-    <xacro:property name="base_height" value="0.1" />
-    <xacro:property name="base_mass" value="10.0" />
-    <xacro:property name="base_length" value="0.8" />
-    <xacro:property name="base_width" value="0.6" />
-    <xacro:property name="wheel_width" value="0.05" />
-    <xacro:property name="wheel_separation" value="0.64" />
-    <xacro:property name="caster_radius" value="0.05" />
-    <xacro:property name="caster_mass" value="0.1" />
-    <xacro:macro name="default_inertial" params="mass">
-        <inertial>
-            <mass value="${mass}" />
-            <inertia ixx="${0.08 * mass}" ixy="0.0" ixz="0.0" iyy="${0.08 * mass}" iyz="0.0" izz="${0.08 * mass}"/>
-        </inertial>
-    </xacro:macro>
-    <link name="base_link">
-        <visual>
-            <origin xyz="0 0 ${wheel_radius + base_height/2}" rpy="0 0 0" />
-            <geometry><box size="${base_length} ${base_width} ${base_height}" /></geometry>
-            <material name="White"><color rgba="1 1 1 1"/></material>
-        </visual>
-        <collision>
-            <origin xyz="0 0 ${wheel_radius + base_height/2}" rpy="0 0 0" />
-            <geometry><box size="${base_length} ${base_width} ${base_height}" /></geometry>
-        </collision>
-        <xacro:default_inertial mass="${base_mass}"/>
-    </link>
-    <xacro:macro name="wheel_link" params="prefix parent_link x_offset y_offset">
-        <link name="${prefix}_wheel_link">
-            <visual>
-                <origin xyz="0 0 0" rpy="1.5708 0 0" />
-                <geometry><cylinder radius="${wheel_radius}" length="${wheel_width}" /></geometry>
-                <material name="Black"><color rgba="0 0 0 1"/></material>
-            </visual>
-            <collision>
-                <origin xyz="0 0 0" rpy="1.5708 0 0" />
-                <geometry><cylinder radius="${wheel_radius}" length="${wheel_width}" /></geometry>
-            </collision>
-            <xacro:default_inertial mass="0.5" />
-        </link>
-        <joint name="${prefix}_wheel_joint" type="continuous">
-            <origin xyz="${x_offset} ${y_offset} ${wheel_radius}" rpy="0 0 0" />
-            <parent link="${parent_link}" />
-            <child link="${prefix}_wheel_link" />
-            <axis xyz="0 1 0" />
-        </joint>
-        <gazebo reference="${prefix}_wheel_link">
-          <material>Gazebo/Black</material>
-        </gazebo>
-    </xacro:macro>
-    <xacro:wheel_link prefix="left" parent_link="base_link" x_offset="0.25" y_offset="${wheel_separation/2}" />
-    <xacro:wheel_link prefix="right" parent_link="base_link" x_offset="0.25" y_offset="-${wheel_separation/2}" />
-    <link name="caster_front_link">
-        <visual>
-            <origin xyz="0 0 0" rpy="0 0 0"/>
-            <geometry><sphere radius="${caster_radius}"/></geometry>
-            <material name="Black"/>
-        </visual>
-        <collision>
-            <origin xyz="0 0 0" rpy="0 0 0"/>
-            <geometry><sphere radius="${caster_radius}"/></geometry>
-        </collision>
-        <xacro:default_inertial mass="${caster_mass}"/>
-    </link>
-    <joint name="caster_front_joint" type="fixed">
-        <origin xyz="${base_length/2 - caster_radius*2} 0 ${caster_radius}" rpy="0 0 0"/>
-        <parent link="base_link" />
-        <child link="caster_front_link" />
-    </joint>
-    <link name="caster_rear_link">
-        <visual>
-            <origin xyz="0 0 0" rpy="0 0 0"/>
-            <geometry><sphere radius="${caster_radius}"/></geometry>
-            <material name="Black"/>
-        </visual>
-        <collision>
-            <origin xyz="0 0 0" rpy="0 0 0"/>
-            <geometry><sphere radius="${caster_radius}"/></geometry>
-        </collision>
-        <xacro:default_inertial mass="${caster_mass}"/>
-    </link>
-    <joint name="caster_rear_joint" type="fixed">
-        <origin xyz="${-base_length/2 + caster_radius*2} 0 ${caster_radius}" rpy="0 0 0"/>
-        <parent link="base_link" />
-        <child link="caster_rear_link" />
-    </joint>
-<xacro:include filename="hybrid_aerial.xacro" />
-    <link name="landing_pad">
-        <visual>
-            <origin xyz="0 0 0" rpy="0 0 0" />
-            <geometry><box size="0.4 0.4 0.01" /></geometry>
-            <material name="Grey"><color rgba="0.5 0.5 0.5 1"/></material>
-        </visual>
-        <collision>
-            <origin xyz="0 0 0" rpy="0 0 0" />
-            <geometry><box size="0.4 0.4 0.01" /></geometry>
-        </collision>
-        <xacro:default_inertial mass="0.1"/>
-    </link>
-    <joint name="landing_pad_joint" type="fixed">
-        <parent link="base_link" />
-        <child link="landing_pad" />
-        <origin xyz="0 0 0.2" rpy="0 0 0" />
-    </joint>
-    <xacro:drone_assembly parent_link="landing_pad" />
-    <ros2_control name="TerrestrialRobot" type="system">
-        <hardware>
-            <plugin>gazebo_ros2_control/GazeboSystem</plugin>
-        </hardware>
-        <joint name="left_wheel_joint">
-            <command_interface name="velocity">
-                <param name="min">-10</param>
-                <param name="max">10</param>
-            </command_interface>
-            <state_interface name="velocity"/>
-            <state_interface name="position"/>
-        </joint>
-        <joint name="right_wheel_joint">
-            <command_interface name="velocity">
-                <param name="min">-10</param>
-                <param name="max">10</param>
-            </command_interface>
-            <state_interface name="velocity"/>
-            <state_interface name="position"/>
-        </joint>
-    </ros2_control>
-    <gazebo>
-        <plugin filename="libgazebo_ros2_control.so" name="gazebo_ros2_control">
-            <parameters>$(find hybrid_robot_description)/config/terrestrial_control.yaml</parameters>
-        </plugin>
-    </gazebo>
-</robot>
+/home/lois/hybrid_robot/hybrid_robot_ws/src/hybrid_robot_description/urdf/hybrid_terrestrial.xacro

Commit message: EL robot puede volar enteramente ahora

File: hybrid_robot_ws/install/hybrid_robot_description/share/hybrid_robot_description/urdf/hybrid_terrestrial.xacro (robot description, xacro)
@@ -1 +1,94 @@
-/home/lois/hybrid_robot/hybrid_robot_ws/src/hybrid_robot_description/urdf/hybrid_terrestrial.xacro
+<?xml version="1.0"?>
+<robot name="hybrid_robot" xmlns:xacro="http://www.ros.org/wiki/xacro">
+    <xacro:property name="wheel_radius" value="0.1" />
+    <xacro:property name="base_height" value="0.1" />
+    <xacro:property name="base_mass" value="5.0" />
+    <xacro:property name="base_length" value="0.8" />
+    <xacro:property name="base_width" value="0.6" />
+    <xacro:property name="wheel_width" value="0.05" />
+    <xacro:property name="wheel_separation" value="0.64" />
+    <xacro:property name="caster_radius" value="0.05" />
+    <xacro:property name="caster_mass" value="0.1" />
+    <xacro:macro name="default_inertial" params="mass">
+        <inertial>
+            <mass value="${mass}" />
+            <inertia ixx="${0.08 * mass}" ixy="0.0" ixz="0.0" iyy="${0.08 * mass}" iyz="0.0" izz="${0.08 * mass}"/>
+        </inertial>
+    </xacro:macro>
+    <link name="base_link">
+        <visual>
+            <origin xyz="0 0 ${wheel_radius + base_height/2}" rpy="0 0 0" />
+            <geometry><box size="${base_length} ${base_width} ${base_height}" /></geometry>
+            <material name="White"><color rgba="1 1 1 1"/></material>
+        </visual>
+        <collision>
+            <origin xyz="0 0 ${wheel_radius + base_height/2}" rpy="0 0 0" />
+            <geometry><box size="${base_length} ${base_width} ${base_height}" /></geometry>
+        </collision>
+        <xacro:default_inertial mass="${base_mass}"/>
+    </link>
+    <xacro:macro name="wheel_link" params="prefix parent_link x_offset y_offset">
+        <link name="${prefix}_wheel_link">
+            <visual>
+                <origin xyz="0 0 0" rpy="1.5708 0 0" />
+                <geometry><cylinder radius="${wheel_radius}" length="${wheel_width}" /></geometry>
+                <material name="Black"><color rgba="0 0 0 1"/></material>
+            </visual>
+            <collision>
+                <origin xyz="0 0 0" rpy="1.5708 0 0" />
+                <geometry><cylinder radius="${wheel_radius}" length="${wheel_width}" /></geometry>
+            </collision>
+            <xacro:default_inertial mass="0.5" />
+        </link>
+        <gazebo reference="${prefix}_wheel_link">
+            <material>Gazebo/Black</material>
+            <mu1 value="1.0"/><mu2 value="1.0"/>
+        </gazebo>
+        <joint name="${prefix}_wheel_joint" type="continuous">
+            <origin xyz="${x_offset} ${y_offset} ${wheel_radius}" rpy="0 0 0" />
+            <parent link="${parent_link}" />
+            <child link="${prefix}_wheel_link" />
+            <axis xyz="0 1 0" />
+        </joint>
+    </xacro:macro>
+    <xacro:wheel_link prefix="left" parent_link="base_link" x_offset="0.25" y_offset="${wheel_separation/2}" />
+    <xacro:wheel_link prefix="right" parent_link="base_link" x_offset="0.25" y_offset="-${wheel_separation/2}" />
+    <link name="caster_front_link">
+        <visual><geometry><sphere radius="${caster_radius}"/></geometry><material name="Black"/></visual>
+        <collision><geometry><sphere radius="${caster_radius}"/></geometry></collision>
+        <xacro:default_inertial mass="${caster_mass}"/>
+    </link>
+    <joint name="caster_front_joint" type="fixed">
+        <origin xyz="${base_length/2 - caster_radius*2} 0 ${caster_radius}" rpy="0 0 0"/>
+        <parent link="base_link" /><child link="caster_front_link" />
+    </joint>
+    <link name="caster_rear_link">
+        <visual><geometry><sphere radius="${caster_radius}"/></geometry><material name="Black"/></visual>
+        <collision><geometry><sphere radius="${caster_radius}"/></geometry></collision>
+        <xacro:default_inertial mass="${caster_mass}"/>
+    </link>
+    <joint name="caster_rear_joint" type="fixed">
+        <origin xyz="${-base_length/2 + caster_radius*2} 0 ${caster_radius}" rpy="0 0 0"/>
+        <parent link="base_link" /><child link="caster_rear_link" />
+    </joint>
+    <link name="landing_pad">
+        <visual>
+            <origin xyz="0 0 0" rpy="0 0 0" />
+            <geometry><box size="0.4 0.4 0.01" /></geometry>
+            <material name="Grey"><color rgba="0.5 0.5 0.5 1"/></material>
+        </visual>
+        <collision>
+            <origin xyz="0 0 0" rpy="0 0 0" />
+            <geometry><box size="0.4 0.4 0.01" /></geometry>
+        </collision>
+        <xacro:default_inertial mass="0.1"/>
+    </link>
+    <joint name="landing_pad_joint" type="fixed">
+        <parent link="base_link" />
+        <child link="landing_pad" />
+        <origin xyz="0 0 0.2" rpy="0 0 0" />
+    </joint>
+    <gazebo reference="base_link">
+        <material>Gazebo/Green</material>
+    </gazebo>
+</robot>

File: hybrid_robot_ws/src/hybrid_robot_description/urdf/hybrid_aerial.xacro (robot description, xacro)
@@ -1,5 +1,5 @@
 <?xml version="1.0"?>
 <robot xmlns:xacro="http://www.ros.org/wiki/xacro">
-    <xacro:macro name="drone_assembly" params="parent_link">
+    <xacro:macro name="drone_assembly">
         <link name="drone_base_link">
             <visual>
@@ -17,12 +17,8 @@
             </inertial>
         </link>
-        <joint name="drone_to_terrestrial_joint" type="fixed">
-            <parent link="${parent_link}" />
-            <child link="drone_base_link" />
-            <origin xyz="0 0 0.01" rpy="0 0 0" />
-        </joint>
         <xacro:macro name="prop" params="p_name x y">
             <link name="${p_name}_link">
                 <visual><geometry><cylinder radius="0.08" length="0.01"/></geometry></visual>
+                <material name="Black"><color rgba="0 0 0 1"/></material>
             </link>
             <joint name="${p_name}_joint" type="fixed">

File: hybrid_robot_ws/src/hybrid_robot_description/urdf/hybrid_terrestrial.xacro (robot description, xacro)
@@ -1,4 +1,4 @@
 <?xml version="1.0"?>
-<robot name="hybrid_robot_terrestrial" xmlns:xacro="http://www.ros.org/wiki/xacro">
+<robot name="hybrid_robot" xmlns:xacro="http://www.ros.org/wiki/xacro">
     <xacro:property name="wheel_radius" value="0.1" />
     <xacro:property name="base_height" value="0.1" />
@@ -28,5 +28,5 @@
         <xacro:default_inertial mass="${base_mass}"/>
     </link>
-  <xacro:macro name="wheel_link" params="prefix parent_link x_offset y_offset">
+    <xacro:macro name="wheel_link" params="prefix parent_link x_offset y_offset">
         <link name="${prefix}_wheel_link">
             <visual>
@@ -42,10 +42,6 @@
         </link>
         <gazebo reference="${prefix}_wheel_link">
-            <mu1 value="1.0"/>
-            <mu2 value="1.0"/>
-            <kp value="10000000.0" />
-            <kd value="1.0" />
-            <fdir1 value="1 0 0"/>
             <material>Gazebo/Black</material>
+            <mu1 value="1.0"/><mu2 value="1.0"/>
         </gazebo>
         <joint name="${prefix}_wheel_joint" type="continuous">
@@ -59,46 +55,21 @@
     <xacro:wheel_link prefix="right" parent_link="base_link" x_offset="0.25" y_offset="-${wheel_separation/2}" />
     <link name="caster_front_link">
-        <visual>
-            <origin xyz="0 0 0" rpy="0 0 0"/>
-            <geometry><sphere radius="${caster_radius}"/></geometry>
-            <material name="Black"/>
-        </visual>
-        <collision>
-            <origin xyz="0 0 0" rpy="0 0 0"/>
-            <geometry><sphere radius="${caster_radius}"/></geometry>
-        </collision>
+        <visual><geometry><sphere radius="${caster_radius}"/></geometry><material name="Black"/></visual>
+        <collision><geometry><sphere radius="${caster_radius}"/></geometry></collision>
         <xacro:default_inertial mass="${caster_mass}"/>
     </link>
     <joint name="caster_front_joint" type="fixed">
         <origin xyz="${base_length/2 - caster_radius*2} 0 ${caster_radius}" rpy="0 0 0"/>
-        <parent link="base_link" />
-        <child link="caster_front_link" />
+        <parent link="base_link" /><child link="caster_front_link" />
     </joint>
     <link name="caster_rear_link">
-        <visual>
-            <origin xyz="0 0 0" rpy="0 0 0"/>
-            <geometry><sphere radius="${caster_radius}"/></geometry>
-            <material name="Black"/>
-        </visual>
-        <collision>
-            <origin xyz="0 0 0" rpy="0 0 0"/>
-            <geometry><sphere radius="${caster_radius}"/></geometry>
-        </collision>
+        <visual><geometry><sphere radius="${caster_radius}"/></geometry><material name="Black"/></visual>
+        <collision><geometry><sphere radius="${caster_radius}"/></geometry></collision>
         <xacro:default_inertial mass="${caster_mass}"/>
     </link>
     <joint name="caster_rear_joint" type="fixed">
         <origin xyz="${-base_length/2 + caster_radius*2} 0 ${caster_radius}" rpy="0 0 0"/>
-        <parent link="base_link" />
-        <child link="caster_rear_link" />
+        <parent link="base_link" /><child link="caster_rear_link" />
     </joint>
-    <gazebo reference="caster_front_link">
-        <mu1 value="0.001"/>
-        <mu2 value="0.001"/>
-    </gazebo>
-    <gazebo reference="caster_rear_link">
-        <mu1 value="0.001"/>
-        <mu2 value="0.001"/>
-    </gazebo>
-<xacro:include filename="hybrid_aerial.xacro" />
     <link name="landing_pad">
         <visual>
@@ -118,31 +89,4 @@
         <origin xyz="0 0 0.2" rpy="0 0 0" />
     </joint>
-    <xacro:drone_assembly parent_link="landing_pad" />
-    <ros2_control name="TerrestrialRobot" type="system">
-        <hardware>
-            <plugin>gazebo_ros2_control/GazeboSystem</plugin>
-        </hardware>
-        <joint name="left_wheel_joint">
-            <command_interface name="velocity">
-                <param name="min">-10</param>
-                <param name="max">10</param>
-            </command_interface>
-            <state_interface name="velocity"/>
-            <state_interface name="position"/>
-        </joint>
-        <joint name="right_wheel_joint">
-            <command_interface name="velocity">
-                <param name="min">-10</param>
-                <param name="max">10</param>
-            </command_interface>
-            <state_interface name="velocity"/>
-            <state_interface name="position"/>
-        </joint>
-    </ros2_control>
-    <gazebo>
-        <plugin filename="libgazebo_ros2_control.so" name="gazebo_ros2_control">
-            <parameters>$(find hybrid_robot_description)/config/terrestrial_control.yaml</parameters>
-        </plugin>
-    </gazebo>
     <gazebo reference="base_link">
         <material>Gazebo/Green</material>
